Commit message: Add files via upload

File: description/robot_base.xacro (robot description, xacro)
@@ -68,5 +68,5 @@
   <link name="chassis">
     <inertial>
-      <mass value="12.0"/>
+      <mass value="2.0"/>
       <origin xyz="0 0 0"/>
       <inertia
@@ -172,5 +172,5 @@
   <link name="caster_link_fl">
     <inertial>
-      <mass value="0.1"/>
+      <mass value="0.01"/>
       <origin xyz="0 0 0"/>
       <inertia ixx="0.012411765597" ixy="-0.000711733678" ixz="0.00050272983" iyy="0.015218160428" iyz="-0.000004273467" izz="0.011763977943"/>
@@ -192,5 +192,5 @@
   <link name="caster_link_fr">
     <inertial>
-      <mass value="0.1"/>
+      <mass value="0.01"/>
       <origin xyz="0 0 0"/>
       <inertia ixx="0.012411765597" ixy="-0.000711733678" ixz="0.00050272983" iyy="0.015218160428" iyz="-0.000004273467" izz="0.011763977943"/>
@@ -212,5 +212,5 @@
   <link name="caster_link_bl">
     <inertial>
-      <mass value="0.3"/>
+      <mass value="0.01"/>
       <origin xyz="0 0 0"/>
       <inertia ixx="0.012411765597" ixy="-0.000711733678" ixz="0.00050272983" iyy="0.015218160428" iyz="-0.000004273467" izz="0.011763977943"/>
@@ -232,5 +232,5 @@
   <link name="caster_link_br">
     <inertial>
-      <mass value="0.3"/>
+      <mass value="0.01"/>
       <origin xyz="0 0 0"/>
       <inertia ixx="0.012411765597" ixy="-0.000711733678" ixz="0.00050272983" iyy="0.015218160428" iyz="-0.000004273467" izz="0.011763977943"/>
@@ -264,5 +264,5 @@
     <inertial>
      <origin xyz="0 0 0" rpy="0 0 0"/>
-     <mass value="0.03"/>
+     <mass value="0.01"/>
             <inertia ixx="${(2/5) * 0.03 * (0.05*0.05)}" ixy="0.0" ixz="0.0"
                     iyy="${(2/5) * 0.03 * (0.05*0.05)}" iyz="0.0"
@@ -272,6 +272,7 @@
 <gazebo reference="front_caster_wheel">
     <material>Gazebo/Grey</material>
-    <mu1 value="0.000001"/> <!-- 摩擦力設定 -->
-    <mu2 value="0.000001"/>
+    <kp value="50000000"/>
+    <mu1 value="0"/> <!-- 摩擦力設定 -->
+    <mu2 value="0"/>
 </gazebo>
 <joint name="back_caster_joint" type="fixed">
@@ -294,5 +295,5 @@
     <inertial>
      <origin xyz="0 0 0" rpy="0 0 0"/>
-     <mass value="0.3"/>
+     <mass value="0.01"/>
             <inertia ixx="${(2/5) * 0.3 * (0.05*0.05)}" ixy="0.0" ixz="0.0"
                     iyy="${(2/5) * 0.3 * (0.05*0.05)}" iyz="0.0"
@@ -302,20 +303,25 @@
 <gazebo reference="back_caster_wheel">
     <material>Gazebo/Grey</material>
-    <mu1 value="0.000001"/> <!-- 摩擦力設定 -->
-    <mu2 value="0.000001"/>
+    <kp value="50000000"/>
+    <mu1 value="0"/> <!-- 摩擦力設定 -->
+    <mu2 value="0"/>
 </gazebo>
 <!-- CASTER WHEEL -->
 <!--gazebo wheels friction -->
 <gazebo reference="left_wheel_joint">
- <mu1 value="1.0"/>
- <mu2 value="1.0"/>
+ <kp value="50000000"/>
+ <kd value="1"/>
+ <mu1 value="1"/>
+ <mu2 value="1"/>
 </gazebo>
 <gazebo reference="right_wheel_joint">
- <mu1 value="1.0"/>
- <mu2 value="1.0"/>
+ <kp value="50000000"/>
+ <kd value="1"/>
+ <mu1 value="1"/>
+ <mu2 value="1"/>
 </gazebo>
 <gazebo reference="chassis">
- <mu1 value="0.0000001"/>
- <mu2 value="0.0000001"/>
+ <mu1 value="0"/>
+ <mu2 value="0"/>
 </gazebo>
 <!--gazebo wheels friction -->
@@ -327,5 +333,5 @@
   <link name="laser_frame" >
     <inertial>
-      <mass value="0.16"/>
+      <mass value="0.001"/>
       <origin rpy="0 0 0" xyz="0 0 0"/>
       <inertia ixx="0.1" ixy="0" ixz="0" iyy="0.1" iyz="0" izz="0.1"/>
@@ -359,6 +365,6 @@
 					</scan>
 					<range>
-						<min>0.05</min>
-						<max>12</max>
+						<min>0.3</min>
+						<max>5.6</max>
 					</range>
 				</ray>
@@ -427,5 +433,5 @@
   <link name="plate_link">
      <inertial>
-      <mass value="20.412"/>
+      <mass value="6"/>
       <origin rpy="0 0 0" xyz="0.01489 0.00213 0.00213"/>
       <inertia ixx="0.003863" ixy="-0.000979" ixz="0.000000" iyy="0.006196" iyz="0.000000" izz="0.006369"/>
@@ -454,5 +460,5 @@
       <!--<origin xyz="0.023 0 0.006" rpy="0 0 0"/>-->
       <origin rpy="0 0 0" xyz="0 0 0"/>
-      <mass value="0.845"/>
+      <mass value="0.08"/>
       <inertia ixx="0.01" ixy="0" ixz="0" iyy="0.01" iyz="0" izz="0.01"/>
     </inertial>
@@ -490,5 +496,5 @@
   <link name="arm_link_1">
     <inertial>
-      <mass value="2.412"/>
+      <mass value="0.02412"/>
       <origin rpy="0 0 0" xyz="0.01489 0.00213 0.00213"/>
       <inertia ixx="0.003863" ixy="-0.000979" ixz="0.000000" iyy="0.006196" iyz="0.000000" izz="0.006369"/>
@@ -520,5 +526,5 @@
   <link name="arm_link_2">
     <inertial>
-      <mass value="1.155"/>
+      <mass value="0.00155"/>
       <origin rpy="0 0 0" xyz="0.10453 0.0017 -0.00297"/>
       <inertia ixx="0.000823" ixy="0.000000" ixz="-0.000000" iyy="0.004447" iyz="0.000000" izz="0.004439"/>
@@ -549,5 +555,5 @@
   <link name="arm_link_3">
     <inertial>
-      <mass value="0.934"/>
+      <mass value="0.00934"/>
       <origin rpy="0 0 0" xyz="0.0001 0.0967 0.02107"/>
       <inertia ixx="0.002459" ixy="0.000000" ixz="0.000000" iyy="0.002571" iyz="-0.000000" izz="0.000535"/>
@@ -579,5 +585,5 @@
   <link name="arm_link_4">
     <inertial>
-      <mass value="0.877"/>
+      <mass value="0.000877"/>
       <origin rpy="0 0 0" xyz="0.00011 0.05103 -0.02319"/>
       <inertia ixx="0.000869" ixy="0.000000" ixz="-0.000000" iyy="0.001173" iyz="-0.000231" izz="0.001091"/>
@@ -609,5 +615,5 @@
   <link name="arm_link_5">
     <inertial>
-      <mass value="0.251"/>
+      <mass value="0.000251"/>
       <origin rpy="0 0 0" xyz="0.0 0.00115 -0.01683"/>
       <inertia ixx="0.000280" ixy="0.000000" ixz="0.000000" iyy="0.000339" iyz="0.000000" izz="0.000119"/>
@@ -629,5 +635,5 @@
   <link name="pen">
     <inertial>
-      <mass value="0.01"/>
+      <mass value="0.00001"/>
       <origin rpy="0 0 0.1" xyz="0.0 0.00115 -0.01683"/>
       <inertia ixx="0.01" ixy="0.000000" ixz="0.000000" iyy="0.01" iyz="0.000000" izz="0.01"/>
